File: _autosave-Project.kicad_sch (KiCad schematic)
At the start: 21 parts, among them P1 USB_C_Plug, SW1 DOUBLE_KEY, U1 MAX15062A, U2 TUSB8041, Y1 24MHz

Commit message: 实现下行USB
Parts:
- added C10, C11, C8, C9: 0.1uF, symbol Lib1:C(MM)-LibCool
- added D1: OVERCUR1, symbol Device:LED
- added D2: OVERCUR2, symbol Device:LED
- added J1, J2: USB3_A, symbol Connector:USB3_A
- added P2: USB_C_Plug, symbol Connector:USB_C_Plug
- added R10, R?: RES(M)-LibCool, symbol Lib1:RES(M)-LibCool
- added R9: 4.7K/5%, symbol Lib1:RES(M)-LibCool
- gave numbers to parts that had none: 4
Connections:
- net +3V3: now also U2.16 (VDD33), U2.26 (USB_SSTXP_DN4), U2.34 (VDD33), U2.52 (VDD33), U2.63 (VDD33), P2.A2 (TX1+), R10.1, R9.1, R?.1
- net GND: now also U2.65 (VSS), D1.1 (K), D2.1 (K)
- net POWER: now also J1.1 (VBUS)
- net at U2.1 (USB_DP_DN1): now also J1.3 (D+)
- net at U2.17 (USB_DP_DN3): now also J2.3 (D+)
- net at U2.18 (USB_DM_DN3): now also J2.2 (D-)
- net at U2.19 (USB_SSTXP_DN3): now also C8.1
- net at U2.2 (USB_DM_DN1): now also J1.2 (D-)
- net at U2.20 (USB_SSTXM_DN3): now also C10.1
- net at U2.22 (USB_SSRXP_DN3): now also J2.6 (SSRX+)
- net at U2.23 (USB_SSRXM_DN3): now also J2.5 (SSRX-)
- net at U2.24 (USB_DP_DN4): now also P2.A6 (D+)
- net at U2.25 (USB_DM_DN4): now also P2.A7 (D-)
- net at U2.27 (USB_SSTXM_DN4): now also P2.A3 (TX1-)
- net at U2.29 (USB_SSRXP_DN4): now also P2.B11 (RX1+)
- net at U2.3 (USB_SSTXP_DN1): now also C9.1
- net at U2.30 (USB_SSRXM_DN4): now also P2.B10 (RX1-)
- net at U2.32 (PWRCTL4/BATEN4): now also R?.2
- net at U2.33 (PWRCTL3/BATEN3): now also R10.2
- net at U2.36 (PWRCTL1/BATEN1): now also R9.2
- net at U2.4 (USB_SSTXM_DN1): now also C11.1
- net at U2.44 (OVERCUR3z): now also D2.2 (A)
- net at U2.46 (OVERCUR1z): now also D1.2 (A)
- net at U2.6 (USB_SSRXP_DN1): now also J1.6 (SSRX+)
- net at U2.7 (USB_SSRXM_DN1): now also J1.5 (SSRX-)
- new net: C11.2, J1.8 (SSTX-)
- new net: C9.2, J1.9 (SSTX+)
- new net: C10.2, J2.8 (SSTX-)
- new net: C8.2, J2.9 (SSTX+)
- new net: P2.A1 (GND), P2.A12 (GND), P2.B1 (GND), P2.B12 (GND)
- new net: P2.A4 (VBUS), P2.A9 (VBUS), P2.B4 (VBUS), P2.B9 (VBUS)
- no-connect marks 0 -> 11
