File: _autosave-Project.kicad_sch (KiCad schematic)
At the start: 45 parts, among them J1 USB3_A, J2 USB3_A, J3 RJ45, P1 USB_C_Plug, P2 USB_C_Plug, SW1 DOUBLE_KEY, U1 MAX15062A, U2 TUSB8041, U3 XR22800, U4 TPS82676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

Commit message: 完成设计
Parts:
- L1: value Inductor-LibCool -> 33uH
Connections:
- no-connect marks 25 -> 40
Changed lines of the file:
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@@
   (junction (at 148.59 25.4) (diameter 0) (color 0 0 0 0)
   )
+  (no_connect (at 207.01 179.07))
+  (no_connect (at 207.01 181.61))
+  (no_connect (at 207.01 186.69))
+  (no_connect (at 207.01 128.27))
+  (no_connect (at 207.01 146.05))
+  (no_connect (at 207.01 143.51))
+  (no_connect (at 207.01 138.43))
+  (no_connect (at 207.01 135.89))
+  (no_connect (at 207.01 130.81))
+  (no_connect (at 184.15 55.88))
+  (no_connect (at 184.15 58.42))
+  (no_connect (at 184.15 60.96))
+  (no_connect (at 184.15 63.5))
+  (no_connect (at 184.15 71.12))
+  (no_connect (at 184.15 73.66))
   (no_connect (at 118.11 86.36))
   (no_connect (at 118.11 93.98))
@@
     )
     (property "Value" "GND-power" (id 1) (at 64.77 173.0471 0)
-      (effects (font (size 1.27 1.27)))
+      (effects (font (size 1.27 1.27)) hide)
     )
     (property "Footprint" "" (id 2) (at 64.77 176.53 0)
@@
       (effects (font (size 1.016 1.016)))
     )
-    (property "Value" "Inductor-LibCool" (id 1) (at 64.77 110.2211 90)
+    (property "Value" "33uH" (id 1) (at 64.77 110.2211 90)
       (effects (font (size 1.016 1.016)))
     )
@@
     )
     (path "/d1e4d07e-dc11-47bf-ba22-d2712be2ec3d"
-      (reference "L1") (unit 1) (value "Inductor-LibCool") (footprint "")
+      (reference "L1") (unit 1) (value "33uH") (footprint "")
     )
     (path "/17dea307-b08f-415f-85dc-aec387c34ccb"
