File: Project.kicad_pcb (KiCad board)
At the start: 0 parts

Commit message: 完成设计
Parts:
- added C1: C_0603_1608Metric, Capacitor_SMD:C_0603_1608Metric, F.Cu at (27.7, 38.4)
- added C10: C_0402_1005Metric, Capacitor_SMD:C_0402_1005Metric, F.Cu at (73.3, 19.9)
- added C11: C_0402_1005Metric, Capacitor_SMD:C_0402_1005Metric, F.Cu at (61.7, 32.9)
- added C14: C_0402_1005Metric, Capacitor_SMD:C_0402_1005Metric, F.Cu at (47.4, 52.3)
- added C15: C_0402_1005Metric, Capacitor_SMD:C_0402_1005Metric, F.Cu at (38.0, 52.3)
- added C16: C_0402_1005Metric, Capacitor_SMD:C_0402_1005Metric, F.Cu at (37.8, 56.4)
- added C2: C_0603_1608Metric, Capacitor_SMD:C_0603_1608Metric, F.Cu at (23.4, 28.3)
- added C3: C_0603_1608Metric, Capacitor_SMD:C_0603_1608Metric, F.Cu at (28.6, 40.0)
- added C4: C_0402_1005Metric, Capacitor_SMD:C_0402_1005Metric, F.Cu at (43.7, 41.4)
- added C5: C_0402_1005Metric, Capacitor_SMD:C_0402_1005Metric, F.Cu at (39.6, 41.4)
- added C8: C_0402_1005Metric, Capacitor_SMD:C_0402_1005Metric, F.Cu at (73.4, 18.0)
- added C9: C_0402_1005Metric, Capacitor_SMD:C_0402_1005Metric, F.Cu at (64.9, 33.5)
- added F1: Fuse_0603_1608Metric, Fuse:Fuse_0603_1608Metric, F.Cu at (27.3, 27.1)
- added J1: USB3_A_Molex_48393-001, Connector_USB:USB3_A_Molex_48393-001, F.Cu at (66.5, 25.8)
- added J2: USB3_A_Molex_48393-001, Connector_USB:USB3_A_Molex_48393-001, F.Cu at (86.7, 25.7)
- added L1: L_0603_1608Metric, Inductor_SMD:L_0603_1608Metric, F.Cu at (33.5, 39.9)
- added P1: USB_C_Receptacle_Amphenol_12401610E4-2A, Connector_USB:USB_C_Receptacle_Amphenol_12401610E4-2A, F.Cu at (21.0, 20.1)
- added R1: R_0402_1005Metric, Resistor_SMD:R_0402_1005Metric, F.Cu at (40.4, 36.6)
- added R12: R_0402_1005Metric, Resistor_SMD:R_0402_1005Metric, F.Cu at (48.6, 52.3)
- added R2: R_0603_1608Metric, Resistor_SMD:R_0603_1608Metric, F.Cu at (31.5, 32.4)
- added R3: R_0402_1005Metric, Resistor_SMD:R_0402_1005Metric, F.Cu at (33.1, 30.6)
- added R4: R_0402_1005Metric, Resistor_SMD:R_0402_1005Metric, F.Cu at (43.4, 34.8)
- added R7: R_0402_1005Metric, Resistor_SMD:R_0402_1005Metric, F.Cu at (32.1, 33.9)
- added R9: R_0402_1005Metric, Resistor_SMD:R_0402_1005Metric, F.Cu at (34.7, 23.2)
- added REF**: USB_C_Receptacle_Amphenol_12401610E4-2A, Connector_USB:USB_C_Receptacle_Amphenol_12401610E4-2A, F.Cu at (48.9, 17.4)
- added REF**: RJ45_Amphenol_RJHSE5380, Connector_RJ:RJ45_Amphenol_RJHSE5380, F.Cu at (22.0, 56.4)
- added SW1: SW_E-Switch_EG1271_DPDT, Button_Switch_THT:SW_E-Switch_EG1271_DPDT, F.Cu at (35.6, 44.9)
- added U1: TDFN-8-1EP_2x2mm_P0.5mm_EP0.8x1.2mm, Package_DFN_QFN:TDFN-8-1EP_2x2mm_P0.5mm_EP0.8x1.2mm, F.Cu at (31.2, 38.0)
- added U2: QFN-64-1EP_8x8mm_P0.4mm_EP6.5x6.5mm_ThermalVias, Package_DFN_QFN:QFN-64-1EP_8x8mm_P0.4mm_EP6.5x6.5mm_ThermalVias, F.Cu at (38.5, 29.7)
- added U3: QFN-32-1EP_5x5mm_P0.5mm_EP3.1x3.1mm_ThermalVias, Package_DFN_QFN:QFN-32-1EP_5x5mm_P0.5mm_EP3.1x3.1mm_ThermalVias, F.Cu at (47.6, 57.0)
- added U4: BGA-9_3x3_2.9x2.35mm, Lib:BGA-9_3x3_2.9x2.35mm, F.Cu at (34.2, 19.7)
- added Y1: OSC_5032, Lib:OSC_5032, F.Cu at (41.5, 40.5)
- added Y2: OSC_5032, Lib:OSC_5032, F.Cu at (42.7, 54.6)
Routing:
- net (no net): track 0.00 -> 1580.9 mm, vias 0 -> 104
Other:
- copper layers 0 -> 2

Commit message: 提交给打样厂
Other:
- board outline added: 81.5 x 53.7 mm
Changed lines of the file:
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@@
       (layerselection 0x00010fc_ffffffff)
       (disableapertmacros false)
-      (usegerberextensions false)
+      (usegerberextensions true)
       (usegerberattributes true)
       (usegerberadvancedattributes true)
@@
       (svgprecision 4)
       (excludeedgelayer true)
-      (plotframeref false)
+      (plotframeref true)
       (viasonmask false)
       (mode 1)
@@
       (sketchpadsonfab false)
       (subtractmaskfromsilk false)
-      (outputformat 1)
+      (outputformat 4)
       (mirror false)
-      (drillshape 1)
+      (drillshape 0)
       (scaleselection 1)
-      (outputdirectory "")
+      (outputdirectory "Gerber/")
     )
   )
@@
     (fp_line (start 2.5 2.5) (end -2.5 2.5)
       (stroke (width 0.1) (type solid)) (layer "F.Fab"))
-    (pad "" smd roundrect (at -0.5 -0.5 270) (size 0.806226 0.806226) (layers "F.Paste") (roundrect_rratio 0.25))
-    (pad "" smd roundrect (at -0.5 0.5 270) (size 0.806226 0.806226) (layers "F.Paste") (roundrect_rratio 0.25))
-    (pad "" smd roundrect (at 0.5 -0.5 270) (size 0.806226 0.806226) (layers "F.Paste") (roundrect_rratio 0.25))
-    (pad "" smd roundrect (at 0.5 0.5 270) (size 0.806226 0.806226) (layers "F.Paste") (roundrect_rratio 0.25))
+    (pad "" smd roundrect (at -0.5 -0.5 270) (size 0.806226 0.806226) (layers "F.Paste") (roundrect_rratio 0.2500006202))
+    (pad "" smd roundrect (at -0.5 0.5 270) (size 0.806226 0.806226) (layers "F.Paste") (roundrect_rratio 0.2500006202))
+    (pad "" smd roundrect (at 0.5 -0.5 270) (size 0.806226 0.806226) (layers "F.Paste") (roundrect_rratio 0.2500006202))
+    (pad "" smd roundrect (at 0.5 0.5 270) (size 0.806226 0.806226) (layers "F.Paste") (roundrect_rratio 0.2500006202))
     (pad "1" smd roundrect (at -2.4375 -1.75 270) (size 0.875 0.25) (layers "F.Cu" "F.Paste" "F.Mask") (roundrect_rratio 0.25))
     (pad "2" smd roundrect (at -2.4375 -1.25 270) (size 0.875 0.25) (layers "F.Cu" "F.Paste" "F.Mask") (roundrect_rratio 0.25))
@@
     (fp_line (start 4 4) (end -4 4)
       (stroke (width 0.1) (type solid)) (layer "F.Fab"))
-    (pad "" smd roundrect (at 0 0 180) (size 1.006976 1.006976) (layers "F.Paste") (roundrect_rratio 0.248268))
+    (pad "" smd roundrect (at 0 0 180) (size 1.006976 1.006976) (layers "F.Paste") (roundrect_rratio 0.2482680819))
     (pad "1" smd roundrect (at -3.95 -3 180) (size 0.8 0.2) (layers "F.Cu" "F.Paste" "F.Mask") (roundrect_rratio 0.25))
     (pad "2" smd roundrect (at -3.95 -2.6 180) (size 0.8 0.2) (layers "F.Cu" "F.Paste" "F.Mask") (roundrect_rratio 0.25))
@@
     )
   )
+  (gr_rect (start 23.622 23.495) (end 23.622 23.622)
+    (stroke (width 0.15) (type default)) (fill none) (layer "B.Adhes"))
+  (gr_rect (start -18.923 -34.417) (end -56.007 -69.596)
+    (stroke (width 0.15) (type default)) (fill none) (layer "B.Adhes"))
+  (gr_rect (start 11.303 11.176) (end 92.837 64.897)
+    (stroke (width 0.1) (type default)) (fill none) (layer "Edge.Cuts"))
   (segment (start 34.163 22.223) (end 34.671 22.731) (width 0.2) (layer "F.Cu") (net 0))
   (segment (start 51.689 21.209) (end 51.816 21.209) (width 0.2) (layer "F.Cu") (net 0))
